File: hardware/Board1.kicad_pcb (KiCad board)
At the start: 2 copper layers, 32.8 x 58.2 mm, 17 parts, among them IC1 AH1912-W-7, J1 DX07S016JA3R1500, J2 Conn_01x04_Pin, J3 Conn_ST_STDC14, SW1 SW_Push, U1 STM32F042G6U6TR, U2 TS2940CW33_RPG, U4 TJA1051T-3

Commit message: Made a few changes regarding STM32
Parts:
- added BT1: XT30, Connector_AMASS:AMASS_XT30PW-M_1x02_P2.50mm_Horizontal, F.Cu at (52.5, 82.1)
- added C3: 4.7n, Capacitor_SMD:C_0603_1608Metric, F.Cu at (40.4, 69.3)
- added D1: D_Schottky, Diode_SMD:D_SOD-123, F.Cu at (60.4, 59.3)
- added D2: D_Schottky, Diode_SMD:D_SOD-123, F.Cu at (60.4, 62.6)
- added D3: D_Schottky, Diode_SMD:D_SOD-123, F.Cu at (60.4, 66.0)
- added J2: USB_C_Receptacle_USB2.0, Connector_USB:USB_C_Receptacle_HRO_TYPE-C-31-M-12, F.Cu at (63.6, 73.8)
- added J4: Conn_01x02_Pin, Connector_JST:JST_EH_S2B-EH_1x02_P2.50mm_Horizontal, F.Cu at (41.9, 65.3)
- added J5: Conn_01x02_Pin, Connector_JST:JST_EH_S2B-EH_1x02_P2.50mm_Horizontal, F.Cu at (51.4, 65.3)
- added R4: 60, Resistor_SMD:R_0603_1608Metric, F.Cu at (40.4, 71.8)
- added R5: 60, Resistor_SMD:R_0603_1608Metric, F.Cu at (40.4, 74.3)
- added R6: 22, Resistor_SMD:R_0603_1608Metric, F.Cu at (40.4, 76.8)
- added R7: 22, Resistor_SMD:R_0603_1608Metric, F.Cu at (40.4, 79.3)
- added R8: 5.1K, Resistor_SMD:R_0603_1608Metric, F.Cu at (40.4, 81.8)
- added R9: 5.1K, Resistor_SMD:R_0603_1608Metric, F.Cu at (40.4, 84.3)
- added U3: STM32F072RBHx, Package_BGA:UFBGA-64_5x5mm_Layout8x8_P0.5mm, F.Cu at (61.8, 82.5)
Connections:
- C1 pad 1: +5V -> 5VA
- IC1 pad 1: +5V -> 5VA
- R1 pad 1: +5V -> 5VA
- U1 pad 17: +3V3 -> +3.3V
- U2 pad 1: +5V -> 5VA
- U4 pad 3: +5V -> 5VA
