File: hardware/vers_2/SpeedCadence.kicad_pcb (KiCad board)
At the start: 2 copper layers, 50 x 31 mm, 41 parts, among them J1 Conn_ST_STDC14, J2 USB_C_Receptacle_USB2.0_16P, J3 Conn_01x03_Pin, J4 Conn_01x02_Pin, J5 Conn_01x04_Pin, J6 Conn_01x02_Pin, SW2 SW_Push, SW3 SW_Push, U2 STM32F103C8Tx, U3 TCAN3414DR, U4 TPSM861253RDXR, Y1 CSTNE8M00G52Z000R0

Commit message: Changed termination on CAN lines from 60 ohm to 120 ohm
Parts:
- removed the C10 at (157.8, 91.2)
- removed the R4 at (160.9, 88.9)
- R3: value 60 -> 120; footprint Resistor_SMD:R_0603_1608Metric -> Resistor_SMD:R_0805_2012Metric
- moved R3 1.76 mm to (162.7, 90.9), turned to -90 degrees
- renumbered C11 to C10, R5 to R4, R6 to R5, R7 to R6, R8 to R7, R9 to R8, R10 to R9
Connections:
- R3 pad 2: Net-(C10-Pad1) -> CANL
Routing:
- net CANL: track 19.7 -> 11.6 mm
- net Net-(C10-Pad1): track 4.82 -> 0.00 mm
- net GND: vias 26 -> 25
Other:
- board text added: "IMPORTANT: Everytime you press the {dblquote}update from PCB{dblquote} button, make sure for U4 to change the net of pad 14 and all the vias to 3.3V, or else the copper pour will not form a connection!"
